File: PCB/MACROPAD.kicad_pcb (KiCad board)
At the start: 2 copper layers, 39.8 x 61.4 mm, 7 parts, among them SW1 SW_Push, SW2 SW_Push, SW3 SW_Push, SW4 SW_Push, U1 XIAO-RP2040-DIP

Commit message: rehecho
Parts:
- added SW5: SW_Push, Button_Switch_Keyboard:SW_Cherry_MX_1.00u_PCB, F.Cu at (187.0, 90.5)
- added SW6: SW_Push, Button_Switch_Keyboard:SW_Cherry_MX_1.00u_PCB, F.Cu at (186.9, 109.6)
Connections:
- U1 pad 6: unconnected-(U1-GPIO7/SCL-Pad6) -> Net-(U1-GPIO7/SCL)
- U1 pad 7: unconnected-(U1-GPIO0/TX-Pad7) -> Net-(U1-GPIO0/TX)
Routing:
- net Net-(U1-GPIO7/SCL): track 0.00 -> 56.8 mm, vias 0 -> 2
- net Net-(U1-GPIO0/TX): track 0.00 -> 56.6 mm, vias 0 -> 4
- net GND: track 93.9 -> 132.1 mm
Other:
- board size 39.8 x 61.4 mm -> 58.8 x 61.4 mm
